Commit message: URSim check: the M1 program runs on a UR10e within 1.4 %
- The UR10e and UR5e descriptions hung the arm from base_link unturned;
  ur_description turns it half a turn (base_link_inertia), so the same
  joint positions pointed the other way. Checked against the UR DH
  parameters and URSim: the tool now stands where the controller has it.
- URScript can number the moves on output register 0, for timing.
- tools/ursim: a small RTDE client and check.py, which runs the M1
  tending program (written by an ignored test) on URSim and compares each
  move's time with KYNEX's plan, blends included: 15.83 s planned against
  16.06 s run.
- The test's teaching turns the arm at its base towards a joint move's
  point first, as someone teaching would, keeping the elbow up.

Co-Authored-By: Claude Opus 5.5 (1M context) <noreply@anthropic.com>

File: apps/kynex/library/ur10e_tending.urdf (robot description, URDF)
Before this commit: robot ur10e, 12 links, 11 joints
Joints:
- joint shoulder_pan_joint: origin xyz=0 0 0.1807 -> xyz=0 0 0.1807 rpy=0 0 3.141592654

File: apps/kynex/library/ur5e.urdf (robot description, URDF)
Before this commit: robot ur5e, 9 links, 8 joints
Joints:
- joint shoulder_pan_joint: origin xyz=0 0 0.1625 -> xyz=0 0 0.1625 rpy=0 0 3.141592654
