Commit message: Library and layout: UR3e and UR16e, a machining centre, snapping, my equipment, measure, report, video
Stage 3, in part: two more UR arms from Universal Robots' own description
(and UR5e's wrist and arm speeds put right at 180°/s), a vertical machining
centre, connectors that snap a robot onto a pedestal or AMR and one conveyor
onto the next, "save as my equipment" for a selected object and its parts,
a two-point ruler, a printable layout report and WebM recording of the view.

Co-Authored-By: Claude Opus 5.5 (1M context) <noreply@anthropic.com>

File: apps/kynex/library/ur5e.urdf (robot description, URDF)
Before this commit: robot ur5e, 9 links, 8 joints
Joints:
- joint elbow_joint: limit lower=-3.1416 upper=3.1416 effort=150 velocity=3.14 -> lower=-3.1416 upper=3.1416 effort=150 velocity=3.1416
- joint shoulder_lift_joint: limit lower=-6.283 upper=6.283 effort=150 velocity=3.14 -> lower=-6.283 upper=6.283 effort=150 velocity=3.1416
- joint shoulder_pan_joint: limit lower=-6.283 upper=6.283 effort=150 velocity=3.14 -> lower=-6.283 upper=6.283 effort=150 velocity=3.1416
- joint wrist_1_joint: limit lower=-6.283 upper=6.283 effort=28 velocity=6.28 -> lower=-6.283 upper=6.283 effort=28 velocity=3.1416
- joint wrist_2_joint: limit lower=-6.283 upper=6.283 effort=28 velocity=6.28 -> lower=-6.283 upper=6.283 effort=28 velocity=3.1416
- joint wrist_3_joint: limit lower=-6.283 upper=6.283 effort=28 velocity=6.28 -> lower=-6.283 upper=6.283 effort=28 velocity=3.1416
