Commit message: Tool catalogue: a gripper, a vacuum plate, a spindle or a torch on any robot
Every robot in the library carries the tool picked for it on its flange:
none, a two-finger gripper, the dual gripper, a vacuum gripper, a deburring
spindle or a welding torch with its gooseneck bent 22°. Grip points arrive
as grippers; a process tool's tip is the robot's TCP. The dual gripper,
once written into each tending robot's URDF, is now the catalogue's, and a
tool changed drops the roles of the grip points that went with it.

Co-Authored-By: Claude Opus 5.5 (1M context) <noreply@anthropic.com>

File: apps/kynex/library/irb1600_tending.urdf (robot description, URDF)
Before this commit: robot irb1600, 12 links, 11 joints
Links:
- removed link grip_a
- removed link grip_b
- removed link gripper
Joints:
- removed joint gripper-grip_a
- removed joint gripper-grip_b
- removed joint tool0-gripper

File: apps/kynex/library/irb1600_track.urdf (robot description, URDF)
Before this commit: robot irb1600_track, 14 links, 13 joints
Links:
- removed link grip_a
- removed link grip_b
- removed link gripper
Joints:
- removed joint gripper-grip_a
- removed joint gripper-grip_b
- removed joint tool0-gripper

File: apps/kynex/library/m1013_tending.urdf (robot description, URDF)
Before this commit: robot m1013, 12 links, 11 joints
Links:
- removed link grip_a
- removed link grip_b
- removed link gripper
Joints:
- removed joint gripper-grip_a
- removed joint gripper-grip_b
- removed joint tool0-gripper

File: apps/kynex/library/ur10e_tending.urdf (robot description, URDF)
Before this commit: robot ur10e, 12 links, 11 joints
Links:
- removed link grip_a
- removed link grip_b
- removed link gripper
Joints:
- removed joint gripper-grip_a
- removed joint gripper-grip_b
- removed joint tool0-gripper
